Commit message: spot micro initial update

File: champ_description/urdf/champ.urdf (robot description, URDF)
Before this commit: robot champ, 29 links, 28 joints
Links:
- link base_link: geometry collision mesh filename=$(find champ_description)/meshes/base_simple.stl scale=0.001 0.001 0.001; visual mesh filename=$(find champ_description)/meshes/base_simple.stl scale=0.001 0.001 0.001
- link camera_link: geometry collision mesh filename=$(find champ_description)/meshes/asus_camera_simple.dae; visual mesh filename=$(find champ_description)/meshes/asus_camera_simple.dae
- link hokuyo_frame: geometry collision box size=0.058 0.058 0.087; visual mesh filename=$(find champ_description)/meshes/hokuyo_utm_30lx.dae
- link lf_hip_link: geometry collision mesh filename=$(find champ_description)/meshes/hip.stl scale=0.001 0.001 0.001; visual mesh filename=$(find champ_description)/meshes/hip.stl scale=0.001 0.001 0.001
- link lf_lower_leg_link: geometry collision mesh filename=$(find champ_description)/meshes/lower_leg_simple.stl scale=0.001 0.001 0.001; visual mesh filename=$(find champ_description)/meshes/lower_leg_simple.stl scale=0.001 0.001 0.001
- link lf_upper_leg_link: geometry collision mesh filename=$(find champ_description)/meshes/upper_leg_simple.stl scale=0.001 0.001 0.001; visual mesh filename=$(find champ_description)/meshes/upper_leg_simple.stl scale=0.001 0.001 0.001
- link lh_hip_link: geometry collision mesh filename=$(find champ_description)/meshes/hip.stl scale=0.001 0.001 0.001; visual mesh filename=$(find champ_description)/meshes/hip.stl scale=0.001 0.001 0.001
- link lh_lower_leg_link: geometry collision mesh filename=$(find champ_description)/meshes/lower_leg_simple.stl scale=0.001 0.001 0.001; visual mesh filename=$(find champ_description)/meshes/lower_leg_simple.stl scale=0.001 0.001 0.001
- link lh_upper_leg_link: geometry collision mesh filename=$(find champ_description)/meshes/upper_leg_simple.stl scale=0.001 0.001 0.001; visual mesh filename=$(find champ_description)/meshes/upper_leg_simple.stl scale=0.001 0.001 0.001
- link rf_hip_link: geometry collision mesh filename=$(find champ_description)/meshes/hip.stl scale=0.001 0.001 0.001; visual mesh filename=$(find champ_description)/meshes/hip.stl scale=0.001 0.001 0.001
- link rf_lower_leg_link: geometry collision mesh filename=$(find champ_description)/meshes/lower_leg_simple.stl scale=0.001 0.001 0.001; visual mesh filename=$(find champ_description)/meshes/lower_leg_simple.stl scale=0.001 0.001 0.001
- link rf_upper_leg_link: geometry collision mesh filename=$(find champ_description)/meshes/upper_leg_simple.stl scale=0.001 0.001 0.001; visual mesh filename=$(find champ_description)/meshes/upper_leg_simple.stl scale=0.001 0.001 0.001
- link rh_hip_link: geometry collision mesh filename=$(find champ_description)/meshes/hip.stl scale=0.001 0.001 0.001; visual mesh filename=$(find champ_description)/meshes/hip.stl scale=0.001 0.001 0.001
- link rh_lower_leg_link: geometry collision mesh filename=$(find champ_description)/meshes/lower_leg_simple.stl scale=0.001 0.001 0.001; visual mesh filename=$(find champ_description)/meshes/lower_leg_simple.stl scale=0.001 0.001 0.001
- link rh_upper_leg_link: geometry collision mesh filename=$(find champ_description)/meshes/upper_leg_simple.stl scale=0.001 0.001 0.001; visual mesh filename=$(find champ_description)/meshes/upper_leg_simple.stl scale=0.001 0.001 0.001
